Commit message: .

File: ros2_ws/src/sebot_description/urdf/mech/mecanum_wheel.urdf.xacro (robot description, xacro)
@@ -27,8 +27,5 @@
         <origin xyz="0 0 0" rpy="0 0 0"/>
         <mass value="${wheel_mass}"/>
-        <inertia
-          ixx="${(wheel_mass/12.0) * (3*wheel_radius*wheel_radius + wheel_width*wheel_width)}" ixy="0" ixz="0"
-          iyy="${(wheel_mass/2.0) * (wheel_radius*wheel_radius)}" iyz="0"
-          izz="${(wheel_mass/12.0) * (3*wheel_radius*wheel_radius + wheel_width*wheel_width)}"/>
+        <inertia ixx="${(wheel_mass/12.0) * (3*wheel_radius*wheel_radius + wheel_width*wheel_width)}" ixy="0" ixz="0" iyy="${(wheel_mass/2.0) * (wheel_radius*wheel_radius)}" iyz="0" izz="${(wheel_mass/12.0) * (3*wheel_radius*wheel_radius + wheel_width*wheel_width)}"/>
       </inertial>
     </link>
@@ -43,18 +40,18 @@
         <friction>
           <ode>
-              <mu>1.0</mu>
-              <mu2>0.0</mu2>
+            <mu>1.0</mu>
+            <mu2>0.0</mu2>
           </ode>
         </friction>
       </surface>
       <visual>
-          <material>
-              <ambient>0.2 0.2 0.2 1.0</ambient>
-              <diffuse>0.2 0.2 0.2 1.0</diffuse>
-              <specular>0.2 0.2 0.2 1.0</specular>
-              <emissive>0.0 0.0 0.0 0.0</emissive>
-          </material>
+        <material>
+          <ambient>0.2 0.2 0.2 1.0</ambient>
+          <diffuse>0.2 0.2 0.2 1.0</diffuse>
+          <specular>0.2 0.2 0.2 1.0</specular>
+          <emissive>0.0 0.0 0.0 0.0</emissive>
+        </material>
       </visual>
-  </gazebo>
+    </gazebo>
   </xacro:macro>
 </robot>

File: ros2_ws/src/sebot_description/urdf/robots/rosmaster_x3.urdf.xacro (robot description, xacro)
@@ -1,65 +1,26 @@
 <?xml version="1.0"?>
 <robot xmlns:xacro="http://www.ros.org/wiki/xacro" name="sebot_description">
-    <xacro:property name="M_PI" value="3.1415926535897931" />
-    <xacro:arg name="robot_name" default="rosmaster_x3"/>
-    <xacro:arg name="prefix" default=""/>
-    <xacro:arg name="use_gazebo" default="false"/>
-    <xacro:include filename="$(find sebot_description)/urdf/mech/rosmaster_x3_base.urdf.xacro"/>
-    <xacro:include filename="$(find sebot_description)/urdf/mech/mecanum_wheel.urdf.xacro"/>
-    <xacro:include filename="$(find sebot_description)/urdf/sensors/rgbd_camera.urdf.xacro"/>
-    <xacro:include filename="$(find sebot_description)/urdf/sensors/lidar.urdf.xacro"/>
-    <xacro:include filename="$(find sebot_description)/urdf/sensors/imu.urdf.xacro"/>
-    <xacro:rosmaster_x3_base prefix="$(arg prefix)"/>
-    <xacro:mecanum_wheel
-      prefix="$(arg prefix)"
-      side="front_left"
-      x_reflect="1"
-      y_reflect="1"/>
-    <xacro:mecanum_wheel
-      prefix="$(arg prefix)"
-      side="front_right"
-      x_reflect="1"
-      y_reflect="-1"/>
-    <xacro:mecanum_wheel
-      prefix="$(arg prefix)"
-      side="back_left"
-      x_reflect="-1"
-      y_reflect="1"/>
-    <xacro:mecanum_wheel
-      prefix="$(arg prefix)"
-      side="back_right"
-      x_reflect="-1"
-      y_reflect="-1"/>
-    <xacro:rgbd_camera
-      prefix="$(arg prefix)"
-      camera_name="cam_1"
-      xyz_offset="0.105 0 0.05"
-      rpy_offset="0 -0.50 0"/>
-    <xacro:lidar_sensor
-      prefix="$(arg prefix)"
-      parent="base_link"
-      frame_id="laser_frame"
-      xyz_offset="0 0 0.0825"
-      rpy_offset="0 0 0"
-      mesh_xyz_offset="0 0 0"
-      mesh_rpy_offset="${-M_PI/2} 0 0"
-      topic_name="scan"/>
-    <xacro:imu_sensor
-      prefix="$(arg prefix)"
-      parent="base_link"
-      frame_id="imu"
-      xyz_offset="0 0 0.006"
-      rpy_offset="0 0 0"
-      update_rate="15.0"
-      topic_name="imu/data"/>
-    <xacro:include filename="$(find sebot_description)/urdf/control/velocity_control_plugin.urdf.xacro" />
-    <xacro:load_velocity_control_plugin use_gazebo="$(arg use_gazebo)"/>
-    <xacro:include filename="$(find sebot_description)/urdf/control/gazebo_sim_ros2_control.urdf.xacro" />
-    <xacro:load_gazebo_sim_ros2_control_plugin
-      robot_name="$(arg robot_name)"
-      use_gazebo="$(arg use_gazebo)"/>
-    <xacro:include filename="$(find sebot_description)/urdf/control/rosmaster_x3_ros2_control.urdf.xacro" />
-    <xacro:yahboom_rosmaster_ros2_control
-      prefix="$(arg prefix)"
-      use_gazebo="$(arg use_gazebo)"/>
+  <xacro:property name="M_PI" value="3.1415926535897931" />
+  <xacro:arg name="robot_name" default="rosmaster_x3"/>
+  <xacro:arg name="prefix" default=""/>
+  <xacro:arg name="use_gazebo" default="false"/>
+  <xacro:include filename="$(find sebot_description)/urdf/mech/rosmaster_x3_base.urdf.xacro"/>
+  <xacro:include filename="$(find sebot_description)/urdf/mech/mecanum_wheel.urdf.xacro"/>
+  <xacro:include filename="$(find sebot_description)/urdf/sensors/rgbd_camera.urdf.xacro"/>
+  <xacro:include filename="$(find sebot_description)/urdf/sensors/lidar.urdf.xacro"/>
+  <xacro:include filename="$(find sebot_description)/urdf/sensors/imu.urdf.xacro"/>
+  <xacro:rosmaster_x3_base prefix="$(arg prefix)"/>
+  <xacro:mecanum_wheel prefix="$(arg prefix)" side="front_left" x_reflect="1" y_reflect="1"/>
+  <xacro:mecanum_wheel prefix="$(arg prefix)" side="front_right" x_reflect="1" y_reflect="-1"/>
+  <xacro:mecanum_wheel prefix="$(arg prefix)" side="back_left" x_reflect="-1" y_reflect="1"/>
+  <xacro:mecanum_wheel prefix="$(arg prefix)" side="back_right" x_reflect="-1" y_reflect="-1"/>
+  <xacro:rgbd_camera prefix="$(arg prefix)" camera_name="cam_1" xyz_offset="0.105 0 0.05" rpy_offset="0 -0.50 0"/>
+  <xacro:lidar_sensor prefix="$(arg prefix)" parent="base_link" frame_id="laser_frame" xyz_offset="0 0 0.0825" rpy_offset="0 0 0" mesh_xyz_offset="0 0 0" mesh_rpy_offset="${-M_PI/2} 0 0" topic_name="scan"/>
+  <xacro:imu_sensor prefix="$(arg prefix)" parent="base_link" frame_id="imu" xyz_offset="0 0 0.006" rpy_offset="0 0 0" update_rate="15.0" topic_name="imu/data"/>
+  <xacro:include filename="$(find sebot_description)/urdf/control/velocity_control_plugin.urdf.xacro" />
+  <xacro:load_velocity_control_plugin use_gazebo="$(arg use_gazebo)"/>
+  <xacro:include filename="$(find sebot_description)/urdf/control/gazebo_sim_ros2_control.urdf.xacro" />
+  <xacro:load_gazebo_sim_ros2_control_plugin robot_name="$(arg robot_name)" use_gazebo="$(arg use_gazebo)"/>
+  <xacro:include filename="$(find sebot_description)/urdf/control/rosmaster_x3_ros2_control.urdf.xacro" />
+  <xacro:yahboom_rosmaster_ros2_control prefix="$(arg prefix)" use_gazebo="$(arg use_gazebo)"/>
 </robot>
