Commit message: update odom node

File: ros2_ws/config/robot.urdf (robot description, URDF)
Before this commit: robot robot model, 4 links, 3 joints
Joints:
- joint base_to_left_wheel: axis (none) -> 0 1 0
- joint base_to_right_wheel: axis (none) -> 0 1 0

Commit message: update: fix odom frame

File: ros2_ws/config/robot.urdf (robot description, URDF)
Before this commit: robot robot_model, 4 links, 3 joints
Links:
- added link caster_wheel; visual sphere radius=0.05
Joints:
- added joint base_to_caster_wheel: type fixed, parent base_link, child caster_wheel, origin xyz=0.2 0 -0.05 rpy=0 0 0

Commit message: update: add gazebo visualization

File: ros2_ws/config/robot.urdf (robot description, URDF)
Before this commit: robot robot_model, 5 links, 4 joints
Links:
- added link imu_link1; visual box size=0.1 0.1 0.05
Joints:
- added joint base_to_imu_link1: type fixed, parent base_link, child imu_link1, origin xyz=0 0 0.1 rpy=0 0 0

Commit message: feat: add uwb transform and update ekf loosele couple and ekf dual

File: ros2_ws/config/robot.urdf (robot description, URDF)
Before this commit: robot robot_model, 6 links, 5 joints
Links:
- link base_link: mass 10.0 -> None; geometry visual box size=0.5 0.3 0.1
- link caster_wheel: mass 0.5 -> None; geometry visual sphere radius=0.05
- link imu_link: mass 0.2 -> None; geometry visual box size=0.1 0.1 0.05
- link left_wheel: mass 1.0 -> None; geometry visual cylinder length=0.05 radius=0.1
- link right_wheel: mass 1.0 -> None; geometry visual cylinder length=0.05 radius=0.1
Joints:
- joint base_footprint_to_base_link: origin xyz=0 0 0.1 rpy=0 0 0 -> xyz=0 0 0.0 rpy=0 0 0
- joint base_to_left_wheel: axis 0 0 1 -> 0 1 0; origin xyz=0 0.15 0 rpy=-1.5708 0 0 -> xyz=0 0.15 0 rpy=-1.57 0 0; type continuous -> fixed
- joint base_to_right_wheel: axis 0 0 1 -> 0 1 0; origin xyz=0 -0.15 0 rpy=-1.5708 0 0 -> xyz=0 -0.15 0 rpy=-1.57 0 0; type continuous -> fixed

Commit message: add: nav2 stack

File: ros2_ws/config/robot.urdf (robot description, URDF)
Before this commit: robot robot_model, 6 links, 5 joints
Links:
- added link laser; visual cylinder length=0.05 radius=0.05
Joints:
- added joint base_to_lidar_link: type fixed, parent base_link, child laser, origin xyz=0 0 0.15 rpy=0 0 0

Commit message: update: localization technology

File: ros2_ws/config/robot.urdf (robot description, URDF)
Before this commit: robot robot_model, 7 links, 6 joints
Links:
- removed link caster_wheel
- added link uwb_link; visual cylinder length=0.04 radius=0.02
- link base_link: geometry visual box size=0.3 0.2 0.08
- link imu_link: geometry visual box size=0.03 0.03 0.01
- link laser: geometry visual cylinder length=0.05 radius=0.03
- link left_wheel: geometry visual cylinder length=0.02 radius=0.0335
- link right_wheel: geometry visual cylinder length=0.02 radius=0.0335
Joints:
- removed joint base_to_caster_wheel
- added joint base_to_uwb_link: type fixed, parent base_link, child uwb_link, origin xyz=0 -0.2 0.0665 rpy=0 0 0
- joint base_footprint_to_base_link: origin xyz=0 0 0.0 rpy=0 0 0 -> xyz=0 0 0.0335 rpy=0 0 0
- joint base_to_imu_link: origin xyz=0 0 0.1 rpy=0 0 0 -> xyz=0 0 0.05 rpy=0 0 0
- joint base_to_left_wheel: axis 0 1 0 -> (none); origin xyz=0 0.15 0 rpy=-1.57 0 0 -> xyz=0 0.1075 0 rpy=-1.5708 0 0
- joint base_to_lidar_link: origin xyz=0 0 0.15 rpy=0 0 0 -> xyz=0.1 0 0.08 rpy=0 0 0
- joint base_to_right_wheel: axis 0 1 0 -> (none); origin xyz=0 -0.15 0 rpy=-1.57 0 0 -> xyz=0 -0.1075 0 rpy=-1.5708 0 0

Commit message: refactor

File: ros2_ws/config/robot.urdf (robot description, URDF)
Before this commit: robot sebot_model, 7 links, 6 joints
Links:
- removed link laser
Joints:
- removed joint base_to_lidar_link
- joint base_to_uwb_link: origin xyz=0 -0.2 0.0665 rpy=0 0 0 -> xyz=0 -0.05 0.0665 rpy=0 0 0
